File: X16-Power-Slab.brd (EAGLE design)
At the start: 152.4 x 63.5 mm, 24 parts, among them J1 CONN_796636-3, J2 CONN_796636-3, J3 CONN_ET60T, U1 LINEAR_AZ1117CR-3.3TRG1DIODES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

Commit message: Updated component values, added test points
Parts:
- C1: value 0.5pF -> 0.47uF; device SparkFun-Capacitors:0402-TIGHT -> SparkFun-Capacitors:0603
- C2: value 0.5pF -> 0.01uF; device SparkFun-Capacitors:0402-TIGHT -> SparkFun-Capacitors:0603
- C3: value 0.1uF -> 10uF
- C4: value 0.1uF -> 22uF
- R1: value (none) -> 1k
- R2: value (none) -> 3.32k
- moved C2 89.0 mm to (-0.85, -283.2)
- moved C1 80.1 mm to (-0.85, -270.5)
Changed lines of the file:
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@@
 <attribute name="PURCHASE-URL" value="https://pricing.snapeda.com/search/part/AZ1117CH-3.3TRG1/?ref=eda" x="-3.81" y="-176.53" size="1.778" layer="27" display="off"/>
 </element>
-<element name="C1" library="SparkFun-Capacitors" library_urn="urn:adsk.eagle:library:510" package="0402-TIGHT" package3d_urn="urn:adsk.eagle:package:41385069/1" value="0.5pF" x="-5.08" y="-190.5" smashed="yes">
-<attribute name="NAME" x="-5.08" y="-189.938" size="0.6096" layer="25" font="vector" ratio="20" align="bottom-center"/>
-<attribute name="PROD_ID" value="CAP-14362" x="-5.08" y="-190.5" size="1.778" layer="27" display="off"/>
-<attribute name="VALUE" x="-5.08" y="-191.062" size="0.6096" layer="27" font="vector" ratio="20" align="top-center"/>
-</element>
-<element name="C2" library="SparkFun-Capacitors" library_urn="urn:adsk.eagle:library:510" package="0402-TIGHT" package3d_urn="urn:adsk.eagle:package:41385069/1" value="0.5pF" x="-5.08" y="-194.31" smashed="yes">
-<attribute name="NAME" x="-5.08" y="-193.748" size="0.6096" layer="25" font="vector" ratio="20" align="bottom-center"/>
-<attribute name="PROD_ID" value="CAP-14362" x="-5.08" y="-194.31" size="1.778" layer="27" display="off"/>
-<attribute name="VALUE" x="-5.08" y="-194.872" size="0.6096" layer="27" font="vector" ratio="20" align="top-center"/>
+<element name="C1" library="SparkFun-Capacitors" library_urn="urn:adsk.eagle:library:510" package="0603" package3d_urn="urn:adsk.eagle:package:41385090/1" value="0.47uF" x="-0.85" y="-270.51" smashed="yes">
+<attribute name="NAME" x="-0.85" y="-269.948" size="0.6096" layer="25" font="vector" ratio="20" align="bottom-center"/>
+<attribute name="PROD_ID" value="CAP-00810" x="-0.85" y="-270.51" size="1.778" layer="27" display="off"/>
+<attribute name="VALUE" value="0.1uF" x="-0.85" y="-271.072" size="0.6096" layer="27" font="vector" ratio="20" align="top-center"/>
+</element>
+<element name="C2" library="SparkFun-Capacitors" library_urn="urn:adsk.eagle:library:510" package="0603" package3d_urn="urn:adsk.eagle:package:41385090/1" value="0.01uF" x="-0.85" y="-283.21" smashed="yes">
+<attribute name="NAME" x="-0.85" y="-282.648" size="0.6096" layer="25" font="vector" ratio="20" align="bottom-center"/>
+<attribute name="PROD_ID" value="CAP-00810" x="-0.85" y="-283.21" size="1.778" layer="27" display="off"/>
+<attribute name="VALUE" value="0.1uF" x="-0.85" y="-283.772" size="0.6096" layer="27" font="vector" ratio="20" align="top-center"/>
 </element>
 <element name="L1" library="SparkFun-Coils" library_urn="urn:adsk.eagle:library:512" package="0806" package3d_urn="urn:adsk.eagle:package:41390597/1" value="2.2μH_SHIELDED_INDUCTOR" x="-81.28" y="-196.85" smashed="yes">
@@
 <attribute name="VALUE" x="-80.01" y="-214.122" size="0.6096" layer="27" font="vector" ratio="20" align="top-center"/>
 </element>
-<element name="R1" library="SparkFun-Resistors" library_urn="urn:adsk.eagle:library:532" package="0603" package3d_urn="urn:adsk.eagle:package:41389018/1" value=" " x="-80.01" y="-217.17" smashed="yes">
+<element name="R1" library="SparkFun-Resistors" library_urn="urn:adsk.eagle:library:532" package="0603" package3d_urn="urn:adsk.eagle:package:41389018/1" value="1k" x="-80.01" y="-217.17" smashed="yes">
 <attribute name="NAME" x="-80.01" y="-216.408" size="0.6096" layer="25" font="vector" ratio="20" align="bottom-center"/>
 <attribute name="PROD_ID" value=" " x="-80.01" y="-217.17" size="1.778" layer="27" display="off"/>
 <attribute name="VALUE" x="-80.01" y="-217.932" size="0.6096" layer="27" font="vector" ratio="20" align="top-center"/>
 </element>
-<element name="R2" library="SparkFun-Resistors" library_urn="urn:adsk.eagle:library:532" package="0603" package3d_urn="urn:adsk.eagle:package:41389018/1" value=" " x="-80.01" y="-220.98" smashed="yes">
+<element name="R2" library="SparkFun-Resistors" library_urn="urn:adsk.eagle:library:532" package="0603" package3d_urn="urn:adsk.eagle:package:41389018/1" value="3.32k" x="-80.01" y="-220.98" smashed="yes">
 <attribute name="NAME" x="-80.01" y="-220.218" size="0.6096" layer="25" font="vector" ratio="20" align="bottom-center"/>
 <attribute name="PROD_ID" value=" " x="-80.01" y="-220.98" size="1.778" layer="27" display="off"/>
@@
 <attribute name="VALUE" x="-81.38" y="-232.426" size="1.27" layer="27" ratio="10"/>
 </element>
-<element name="C3" library="SparkFun-Capacitors" library_urn="urn:adsk.eagle:library:510" package="0603" package3d_urn="urn:adsk.eagle:package:41385090/1" value="0.1uF" x="-80.01" y="-234.95" smashed="yes">
+<element name="C3" library="SparkFun-Capacitors" library_urn="urn:adsk.eagle:library:510" package="0603" package3d_urn="urn:adsk.eagle:package:41385090/1" value="10uF" x="-80.01" y="-234.95" smashed="yes">
 <attribute name="NAME" x="-80.01" y="-234.188" size="0.6096" layer="25" font="vector" ratio="20" align="bottom-center"/>
 <attribute name="PROD_ID" value="CAP-00810" x="-80.01" y="-234.95" size="1.778" layer="27" display="off"/>
 <attribute name="VALUE" x="-80.01" y="-235.712" size="0.6096" layer="27" font="vector" ratio="20" align="top-center"/>
 </element>
-<element name="C4" library="SparkFun-Capacitors" library_urn="urn:adsk.eagle:library:510" package="0603" package3d_urn="urn:adsk.eagle:package:41385090/1" value="0.1uF" x="-80.01" y="-238.76" smashed="yes">
+<element name="C4" library="SparkFun-Capacitors" library_urn="urn:adsk.eagle:library:510" package="0603" package3d_urn="urn:adsk.eagle:package:41385090/1" value="22uF" x="-80.01" y="-238.76" smashed="yes">
 <attribute name="NAME" x="-80.01" y="-237.998" size="0.6096" layer="25" font="vector" ratio="20" align="bottom-center"/>
 <attribute name="PROD_ID" value="CAP-00810" x="-80.01" y="-238.76" size="1.778" layer="27" display="off"/>
@@
 <contactref element="U$2" pad="PIN3"/>
 <contactref element="C2" pad="1"/>
-<wire x1="16.51" y1="-176.53" x2="-5.58" y2="-194.31" width="0" layer="19" extent="1-1"/>
+<wire x1="-1.7" y1="-283.21" x2="16.51" y2="-176.53" width="0" layer="19" extent="1-1"/>
 </signal>
 <signal name="N$2">
@@
 <contactref element="C2" pad="2"/>
 <contactref element="U$3" pad="C"/>
-<wire x1="16.51" y1="-179.07" x2="-4.58" y2="-194.31" width="0" layer="19" extent="1-1"/>
-<wire x1="-82.18" y1="-196.85" x2="-4.58" y2="-194.31" width="0" layer="19" extent="1-1"/>
+<wire x1="-82.18" y1="-196.85" x2="16.51" y2="-179.07" width="0" layer="19" extent="1-1"/>
 <wire x1="-80.79" y1="-229.87" x2="-82.18" y2="-196.85" width="0" layer="19" extent="1-1"/>
+<wire x1="0" y1="-283.21" x2="-80.79" y2="-229.87" width="0" layer="19" extent="1-1"/>
 </signal>
 <signal name="N$4">
@@
 <contactref element="C9" pad="+"/>
 <contactref element="U$2" pad="PIN2"/>
-<wire x1="16.51" y1="-177.8" x2="-5.58" y2="-190.5" width="0" layer="19" extent="1-1"/>
-<wire x1="-79.16" y1="-213.36" x2="-5.58" y2="-190.5" width="0" layer="19" extent="1-1"/>
+<wire x1="-1.7" y1="-270.51" x2="16.51" y2="-177.8" width="0" layer="19" extent="1-1"/>
+<wire x1="-79.16" y1="-213.36" x2="-1.7" y2="-270.51" width="0" layer="19" extent="1-1"/>
 </signal>
 <signal name="GND/2.2D">
@@
 <contactref element="U$2" pad="PIN4"/>
 <contactref element="U$3" pad="A"/>
-<wire x1="6.315" y1="-175.26" x2="-4.58" y2="-190.5" width="0" layer="19" extent="1-1"/>
 <wire x1="16.51" y1="-175.26" x2="6.315" y2="-175.26" width="0" layer="19" extent="1-1"/>
-<wire x1="-80.86" y1="-201.93" x2="-4.58" y2="-190.5" width="0" layer="19" extent="1-1"/>
+<wire x1="-80.86" y1="-201.93" x2="6.315" y2="-175.26" width="0" layer="19" extent="1-1"/>
 <wire x1="-80.86" y1="-205.74" x2="-80.86" y2="-201.93" width="0" layer="19" extent="1-1"/>
 <wire x1="-80.86" y1="-209.55" x2="-80.86" y2="-205.74" width="0" layer="19" extent="1-1"/>
@@
 <wire x1="-80.86" y1="-224.79" x2="-80.86" y2="-213.36" width="0" layer="19" extent="1-1"/>
 <wire x1="-76.69" y1="-229.87" x2="-80.86" y2="-224.79" width="0" layer="19" extent="1-1"/>
+<wire x1="0" y1="-270.51" x2="-76.69" y2="-229.87" width="0" layer="19" extent="1-1"/>
 </signal>
 <signal name="GND">

Commit message: Updated reverse voltage protection
Parts:
- added D2: 12V, SparkFun-LED:LED-0603
- added D3: 5.2V, SparkFun-LED:LED-0603
- added D4: 3.3V, SparkFun-LED:LED-0603
- added DIODE: 40V, X15-Conversion-Parts-Library:DO214AC
- added R5: 600, SparkFun-Resistors:0603
- added R6: 300, SparkFun-Resistors:0603
- added R7: 200, SparkFun-Resistors:0603
- added U$4: (no value), X15-Conversion-Parts-Library:5.2V_TESTPOINT
- added U$5: (no value), X15-Conversion-Parts-Library:12V_TESTPOINT
- CIN1: value 10uF -> 180uF
- COUT1, COUT2, COUT3: value 10uF -> 150uF
- L1: value 2.2μH_SHIELDED_INDUCTOR -> 15uH
- U$3: value CDBG520-G -> (none); device X15-Conversion-Parts-Library:DO214AC -> X15-Conversion-Parts-Library:3.3V_TESTPOINT
- moved U$3 284.0 mm to (31.8, 31.8)
- renumbered C1 to CIN2, C6 to COUT1, C7 to COUT2, C8 to COUT3, C9 to CIN1
Connections:
- net GND/2.2D: now also DIODE.A; no longer U$3.A
- net N$2: now also DIODE.C; no longer U$3.C
