File: X16_PowerSlab_V2.sch (EAGLE design)
At the start: 39 parts, among them J4 796636-6

Commit message: fixed a resistor value
Parts:
- R1: value (none) -> 1k
- R2: value (none) -> 3.32k
- R4: value (none) -> 1M
Changed lines of the file:
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@@
 <part name="CIN2" library="SparkFun-Capacitors" library_urn="urn:adsk.eagle:library:510" deviceset="0.1UF" device="-0603-25V-(+80/-20%)" package3d_urn="urn:adsk.eagle:package:41385090/1" value="0.47uF"/>
 <part name="C2" library="SparkFun-Capacitors" library_urn="urn:adsk.eagle:library:510" deviceset="0.1UF" device="-0603-25V-(+80/-20%)" package3d_urn="urn:adsk.eagle:package:41385090/1" value="0.01uF"/>
-<part name="R1" library="SparkFun-Resistors" library_urn="urn:adsk.eagle:library:532" deviceset="RESISTOR" device="0603" package3d_urn="urn:adsk.eagle:package:41389018/1" value=" "/>
-<part name="R2" library="SparkFun-Resistors" library_urn="urn:adsk.eagle:library:532" deviceset="RESISTOR" device="0603" package3d_urn="urn:adsk.eagle:package:41389018/1" value=" "/>
+<part name="R1" library="SparkFun-Resistors" library_urn="urn:adsk.eagle:library:532" deviceset="RESISTOR" device="0603" package3d_urn="urn:adsk.eagle:package:41389018/1" value="1k"/>
+<part name="R2" library="SparkFun-Resistors" library_urn="urn:adsk.eagle:library:532" deviceset="RESISTOR" device="0603" package3d_urn="urn:adsk.eagle:package:41389018/1" value="3.32k"/>
 <part name="RADJ" library="SparkFun-Resistors" library_urn="urn:adsk.eagle:library:532" deviceset="RESISTOR" device="0603" package3d_urn="urn:adsk.eagle:package:41389018/1" value=" "/>
 <part name="40V_DIODE" library="X15-Conversion-Parts-Library" deviceset="CDBG520-G" device="" value="40V"/>
@@
 <part name="BACKPLANE_CONN" library="X16_Power_Slab" deviceset="CONN_ET60T" device="" package3d_urn="urn:adsk.eagle:package:41523995/2"/>
 <part name="D1" library="SparkFun-DiscreteSemi" library_urn="urn:adsk.eagle:library:514" deviceset="DIODE-ZENER" device="-BZT52C3V6S" package3d_urn="urn:adsk.eagle:package:38441/2" value="3.6V"/>
-<part name="R4" library="SparkFun-Resistors" library_urn="urn:adsk.eagle:library:532" deviceset="RESISTOR" device="0603" package3d_urn="urn:adsk.eagle:package:41389018/1" value=" "/>
+<part name="R4" library="SparkFun-Resistors" library_urn="urn:adsk.eagle:library:532" deviceset="RESISTOR" device="0603" package3d_urn="urn:adsk.eagle:package:41389018/1" value="1M"/>
 <part name="TRANS_REVERSE_VOLT_PROTEC" library="X15_Brickstribution" deviceset="TRANS_IRF1018ESTRLPBF" device="" package3d_urn="urn:adsk.eagle:package:25914649/1"/>
 <part name="R8" library="SparkFun-Resistors" library_urn="urn:adsk.eagle:library:532" deviceset="0.1OHM" device="-0603-1/3W-1%" package3d_urn="urn:adsk.eagle:package:41389018/1" value="0.1"/>

Commit message: Minh Update
Parts:
- removed D2: 12V, SparkFun-LED:LED-RED-0805
- removed D3: 5.2V, SparkFun-LED:LED-RED-0805
- removed R5, R6: (no value), SparkFun-Resistors:RESISTOR0603
- C2: value 0.01uF -> 0.1uF
- CIN2: value 0.47uF -> 0.1uF
- renumbered 12V_TP to 12V, 48V_GND_TP to 48V_GND, 48V_TP to 48V, 5.2V_TP to 5.2V, D6 to 12V_LED, D7 to 5.2V_LED, GND_TP to GND
Connections:
- removed net N$3: D2.A, R5.2
- removed net N$5: D3.A, R6.2
- net 12V: no longer R5.1
- net 5.2V: no longer R6.1
- net GND: no longer D2.C, D3.C
Other:
- note removed: "LED Voltage Tests"

Commit message: Minh Update 3
Parts:
- added R3: 150k, SparkFun-Resistors:0.1OHM-0603-1/3W-1%
- added R5: 220k, SparkFun-Resistors:0.1OHM-0603-1/3W-1%
- R10: value 0.1 -> 250
- R8: value 0.1 -> 10k
- R9: value 0.1 -> 500
Connections:
- removed net PMBUS_GND: BACKPLANE_CONN.22, BMR480_POWERBRICK.PMBUS_GND
- net GND: now also BACKPLANE_CONN.22, BMR480_POWERBRICK.PMBUS_GND, R3.2, R5.2
- net PMBUS_SA0: now also R3.1; no longer BACKPLANE_CONN.17
- net PMBUS_SA1: now also R5.1; no longer BACKPLANE_CONN.18
Changed lines of the file:
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@@
 <part name="R4" library="SparkFun-Resistors" library_urn="urn:adsk.eagle:library:532" deviceset="RESISTOR" device="0603" package3d_urn="urn:adsk.eagle:package:41389018/1" value="1M"/>
 <part name="TRANS_REVERSE_VOLT_PROTEC" library="X15_Brickstribution" deviceset="TRANS_IRF1018ESTRLPBF" device="" package3d_urn="urn:adsk.eagle:package:25914649/1"/>
-<part name="R8" library="SparkFun-Resistors" library_urn="urn:adsk.eagle:library:532" deviceset="0.1OHM" device="-0603-1/3W-1%" package3d_urn="urn:adsk.eagle:package:41389018/1" value="0.1"/>
-<part name="R9" library="SparkFun-Resistors" library_urn="urn:adsk.eagle:library:532" deviceset="0.1OHM" device="-0603-1/3W-1%" package3d_urn="urn:adsk.eagle:package:41389018/1" value="0.1"/>
-<part name="R10" library="SparkFun-Resistors" library_urn="urn:adsk.eagle:library:532" deviceset="0.1OHM" device="-0603-1/3W-1%" package3d_urn="urn:adsk.eagle:package:41389018/1" value="0.1"/>
+<part name="R8" library="SparkFun-Resistors" library_urn="urn:adsk.eagle:library:532" deviceset="0.1OHM" device="-0603-1/3W-1%" package3d_urn="urn:adsk.eagle:package:41389018/1" value="10k"/>
+<part name="R9" library="SparkFun-Resistors" library_urn="urn:adsk.eagle:library:532" deviceset="0.1OHM" device="-0603-1/3W-1%" package3d_urn="urn:adsk.eagle:package:41389018/1" value="500"/>
+<part name="R10" library="SparkFun-Resistors" library_urn="urn:adsk.eagle:library:532" deviceset="0.1OHM" device="-0603-1/3W-1%" package3d_urn="urn:adsk.eagle:package:41389018/1" value="250"/>
 <part name="D5" library="SparkFun-LED" library_urn="urn:adsk.eagle:library:529" deviceset="LED-RED" device="-0805" package3d_urn="urn:adsk.eagle:package:41389318/1" value="48V"/>
 <part name="12V_LED" library="SparkFun-LED" library_urn="urn:adsk.eagle:library:529" deviceset="LED-RED" device="-0805" package3d_urn="urn:adsk.eagle:package:41389318/1" value="12V"/>
@@
 <part name="48V_GND" library="X16-ExtraComponents" deviceset="TESTPOINT_5.04MM" device=""/>
 <part name="GND" library="X16-ExtraComponents" deviceset="TESTPOINT_5.04MM" device=""/>
+<part name="R3" library="SparkFun-Resistors" library_urn="urn:adsk.eagle:library:532" deviceset="0.1OHM" device="-0603-1/3W-1%" package3d_urn="urn:adsk.eagle:package:41389018/1" value="150k"/>
+<part name="R5" library="SparkFun-Resistors" library_urn="urn:adsk.eagle:library:532" deviceset="0.1OHM" device="-0603-1/3W-1%" package3d_urn="urn:adsk.eagle:package:41389018/1" value="220k"/>
 </parts>
 <sheets>
@@
 <attribute name="NAME" x="138.43" y="23.876" size="1.778" layer="95"/>
 </instance>
+<instance part="R3" gate="G$1" x="38.1" y="76.2" smashed="yes">
+<attribute name="NAME" x="38.1" y="77.724" size="1.778" layer="95" font="vector" align="bottom-center"/>
+<attribute name="VALUE" x="38.1" y="74.676" size="1.778" layer="96" font="vector" align="top-center"/>
+</instance>
+<instance part="R5" gate="G$1" x="38.1" y="63.5" smashed="yes">
+<attribute name="NAME" x="38.1" y="65.024" size="1.778" layer="95" font="vector" align="bottom-center"/>
+<attribute name="VALUE" x="38.1" y="61.976" size="1.778" layer="96" font="vector" align="top-center"/>
+</instance>
 </instances>
 <busses>
@@
 <label x="157.48" y="22.86" size="1.778" layer="95"/>
 </segment>
+<segment>
+<label x="55.88" y="154.94" size="1.778" layer="95"/>
+<pinref part="BMR480_POWERBRICK" gate="G$1" pin="PMBUS_GND"/>
+<wire x1="53.34" y1="154.94" x2="55.88" y2="154.94" width="0.1524" layer="91"/>
+</segment>
+<segment>
+<pinref part="BACKPLANE_CONN" gate="G$1" pin="22"/>
+<wire x1="256.54" y1="119.38" x2="264.16" y2="119.38" width="0.1524" layer="91"/>
+<label x="256.54" y="119.38" size="1.778" layer="95"/>
+</segment>
+<segment>
+<pinref part="R3" gate="G$1" pin="2"/>
+<wire x1="43.18" y1="76.2" x2="55.88" y2="76.2" width="0.1524" layer="91"/>
+<label x="50.8" y="76.2" size="1.778" layer="95"/>
+</segment>
+<segment>
+<pinref part="R5" gate="G$1" pin="2"/>
+<wire x1="43.18" y1="63.5" x2="55.88" y2="63.5" width="0.1524" layer="91"/>
+<label x="50.8" y="63.5" size="1.778" layer="95"/>
+</segment>
 </net>
 <net name="48V_GND" class="0">
@@
 </segment>
 </net>
-<net name="PMBUS_GND" class="0">
-<segment>
-<label x="55.88" y="154.94" size="1.778" layer="95"/>
-<pinref part="BMR480_POWERBRICK" gate="G$1" pin="PMBUS_GND"/>
-<wire x1="53.34" y1="154.94" x2="55.88" y2="154.94" width="0.1524" layer="91"/>
-</segment>
-<segment>
-<pinref part="BACKPLANE_CONN" gate="G$1" pin="22"/>
-<wire x1="256.54" y1="119.38" x2="264.16" y2="119.38" width="0.1524" layer="91"/>
-<label x="256.54" y="119.38" size="1.778" layer="95"/>
-</segment>
-</net>
 <net name="PMBUS_SDA" class="0">
 <segment>
@@
 </segment>
 <segment>
-<pinref part="BACKPLANE_CONN" gate="G$1" pin="18"/>
-<wire x1="256.54" y1="129.54" x2="264.16" y2="129.54" width="0.1524" layer="91"/>
-<label x="256.54" y="129.54" size="1.778" layer="95"/>
+<pinref part="R5" gate="G$1" pin="1"/>
+<wire x1="33.02" y1="63.5" x2="17.78" y2="63.5" width="0.1524" layer="91"/>
+<label x="17.78" y="63.5" size="1.778" layer="95"/>
 </segment>
 </net>
@@
 </segment>
 <segment>
-<pinref part="BACKPLANE_CONN" gate="G$1" pin="17"/>
-<wire x1="256.54" y1="132.08" x2="264.16" y2="132.08" width="0.1524" layer="91"/>
-<label x="256.54" y="132.08" size="1.778" layer="95"/>
-</segment>
-</net>
+<pinref part="R3" gate="G$1" pin="1"/>
+<wire x1="33.02" y1="76.2" x2="17.78" y2="76.2" width="0.1524" layer="91"/>
+<label x="17.78" y="76.2" size="1.778" layer="95"/>
+</segment>
+</net>
