File: X16_PowerSlab_V2.sch (EAGLE design)
At the start: 37 parts, among them J4 796636-6

Commit message: Minh update 4
Parts:
- CIN1: value 150uF -> 594D187X0016R2T; device X15-Conversion-Parts-Library:C-TANTALUM(10UF_150UF) -> X16_Power_Slab:594D187X0016R2T
Connections:
- net GND: now also CIN1.2; no longer CIN1.-
- net VIN: now also CIN1.1; no longer CIN1.+
Changed lines of the file:
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@@
 <part name="COUT5" library="X15-Conversion-Parts-Library" deviceset="C-TANTALUM(10UF_150UF)" device="" package3d_urn="urn:adsk.eagle:package:25131320/3" value="150uF"/>
 <part name="COUT6" library="X15-Conversion-Parts-Library" deviceset="C-TANTALUM(10UF_150UF)" device="" package3d_urn="urn:adsk.eagle:package:25131320/3" value="150uF"/>
-<part name="CIN1" library="X15-Conversion-Parts-Library" deviceset="C-TANTALUM(10UF_150UF)" device="" package3d_urn="urn:adsk.eagle:package:25131320/3" value="150uF"/>
 <part name="CR2" library="X16_Power_Slab" deviceset="RBS2MM40CTR" device=""/>
 <part name="48V" library="X16-ExtraComponents" deviceset="TESTPOINT_5.04MM" device="" value="48V"/>
@@
 <part name="R3" library="SparkFun-Resistors" library_urn="urn:adsk.eagle:library:532" deviceset="0.1OHM" device="-0603-1/3W-1%" package3d_urn="urn:adsk.eagle:package:41389018/1" value="150k"/>
 <part name="R5" library="SparkFun-Resistors" library_urn="urn:adsk.eagle:library:532" deviceset="0.1OHM" device="-0603-1/3W-1%" package3d_urn="urn:adsk.eagle:package:41389018/1" value="220k"/>
+<part name="CIN1" library="X16_Power_Slab" deviceset="594D187X0016R2T" device=""/>
 </parts>
 <sheets>
@@
 <attribute name="VALUE" x="82.296" y="46.609" size="0.762" layer="96"/>
 </instance>
-<instance part="CIN1" gate="G$1" x="-60.96" y="66.04" smashed="yes">
-<attribute name="NAME" x="-59.944" y="66.675" size="0.762" layer="95"/>
-<attribute name="VALUE" x="-59.944" y="61.849" size="0.762" layer="96"/>
-</instance>
 <instance part="CR2" gate="A" x="-73.66" y="71.12" smashed="yes">
 <attribute name="VALUE" x="-77.5462" y="65.5828" size="3.4798" layer="96" ratio="10" rot="SR0"/>
 <attribute name="NAME" x="-76.4794" y="73.8124" size="3.4798" layer="95" ratio="10" rot="SR0"/>
+</instance>
+<instance part="CIN1" gate="A" x="-60.96" y="68.58" smashed="yes" rot="R270">
+<attribute name="VALUE" x="-84.2772" y="58.4962" size="3.4798" layer="96" ratio="10" rot="SR270" display="off"/>
+<attribute name="NAME" x="-67.5894" y="57.9628" size="3.4798" layer="95" ratio="10" rot="SR0"/>
 </instance>
 </instances>
@@
 <pinref part="COUT5" gate="G$1" pin="-"/>
 <pinref part="COUT6" gate="G$1" pin="-"/>
-<pinref part="CIN1" gate="G$1" pin="-"/>
+<pinref part="CIN1" gate="A" pin="2"/>
 </segment>
 </net>
@@
 <junction x="-48.26" y="71.12"/>
 <wire x1="-48.26" y1="71.12" x2="-15.24" y2="71.12" width="0.1524" layer="91"/>
-<pinref part="CIN1" gate="G$1" pin="+"/>
 <pinref part="CR2" gate="A" pin="1"/>
 <wire x1="-63.5" y1="71.12" x2="-60.96" y2="71.12" width="0.1524" layer="91"/>
 <junction x="-60.96" y="71.12"/>
-</segment>
-</net>
+<pinref part="CIN1" gate="A" pin="1"/>
+</segment>
+</net>

Commit message: Minh Update 5
Parts:
- removed D5: 48V, SparkFun-LED:LED-RED-0805
- added 48V_LED: 48V, led:LEDCHIPLED_0805
- 12V_LED, 5.2V_LED: device SparkFun-LED:LED-RED-0805 -> led:LEDCHIPLED_0805
- D1: value 3.6V -> PZU15B3A,115
Connections:
- net 48V_GND: now also 48V_LED.C; no longer D5.C
- net 5.2V: now also BACKPLANE_CONN.P07, BACKPLANE_CONN.P08; no longer BACKPLANE_CONN.P05, BACKPLANE_CONN.P06
- net GND: now also BACKPLANE_CONN.P05, BACKPLANE_CONN.P06; no longer BACKPLANE_CONN.P07, BACKPLANE_CONN.P08
- net N$9: now also 48V_LED.A; no longer D5.A
Changed lines of the file:
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@@
 <part name="FRAME1" library="SparkFun-Aesthetics" library_urn="urn:adsk.eagle:library:507" deviceset="FRAME-A4L" device=""/>
 <part name="BACKPLANE_CONN" library="X16_Power_Slab" deviceset="CONN_ET60T" device="" package3d_urn="urn:adsk.eagle:package:41523995/2"/>
-<part name="D1" library="SparkFun-DiscreteSemi" library_urn="urn:adsk.eagle:library:514" deviceset="DIODE-ZENER" device="-BZT52C3V6S" package3d_urn="urn:adsk.eagle:package:38441/2" value="3.6V"/>
+<part name="D1" library="SparkFun-DiscreteSemi" library_urn="urn:adsk.eagle:library:514" deviceset="DIODE-ZENER" device="-BZT52C3V6S" package3d_urn="urn:adsk.eagle:package:38441/2" value="PZU15B3A,115"/>
 <part name="R4" library="SparkFun-Resistors" library_urn="urn:adsk.eagle:library:532" deviceset="RESISTOR" device="0603" package3d_urn="urn:adsk.eagle:package:41389018/1" value="1M"/>
 <part name="TRANS_REVERSE_VOLT_PROTEC" library="X15_Brickstribution" deviceset="TRANS_IRF1018ESTRLPBF" device="" package3d_urn="urn:adsk.eagle:package:25914649/1"/>
@@
 <part name="R9" library="SparkFun-Resistors" library_urn="urn:adsk.eagle:library:532" deviceset="0.1OHM" device="-0603-1/3W-1%" package3d_urn="urn:adsk.eagle:package:41389018/1" value="500"/>
 <part name="R10" library="SparkFun-Resistors" library_urn="urn:adsk.eagle:library:532" deviceset="0.1OHM" device="-0603-1/3W-1%" package3d_urn="urn:adsk.eagle:package:41389018/1" value="250"/>
-<part name="D5" library="SparkFun-LED" library_urn="urn:adsk.eagle:library:529" deviceset="LED-RED" device="-0805" package3d_urn="urn:adsk.eagle:package:41389318/1" value="48V"/>
-<part name="12V_LED" library="SparkFun-LED" library_urn="urn:adsk.eagle:library:529" deviceset="LED-RED" device="-0805" package3d_urn="urn:adsk.eagle:package:41389318/1" value="12V"/>
-<part name="5.2V_LED" library="SparkFun-LED" library_urn="urn:adsk.eagle:library:529" deviceset="LED-RED" device="-0805" package3d_urn="urn:adsk.eagle:package:41389318/1" value="5.2V"/>
+<part name="48V_LED" library="led" library_urn="urn:adsk.eagle:library:259" deviceset="LED" device="CHIPLED_0805" package3d_urn="urn:adsk.eagle:package:15821/2" value="48V"/>
+<part name="12V_LED" library="led" library_urn="urn:adsk.eagle:library:259" deviceset="LED" device="CHIPLED_0805" package3d_urn="urn:adsk.eagle:package:15821/2" value="12V"/>
+<part name="5.2V_LED" library="led" library_urn="urn:adsk.eagle:library:259" deviceset="LED" device="CHIPLED_0805" package3d_urn="urn:adsk.eagle:package:15821/2" value="5.2V"/>
 <part name="BMR480_POWERBRICK" library="X16_Power_Slab" deviceset="CONN_BMR480_BRICK" device=""/>
 <part name="BACK_EMF" library="X16_Power_Slab" deviceset="SMBJ12CA" device=""/>
@@
 <attribute name="VALUE" x="99.06" y="44.196" size="1.778" layer="96" font="vector" align="top-center"/>
 </instance>
-<instance part="D5" gate="G$1" x="111.76" y="71.12" smashed="yes" rot="R90">
+<instance part="48V_LED" gate="G$1" x="111.76" y="71.12" smashed="yes" rot="R90">
 <attribute name="NAME" x="116.332" y="67.691" size="1.778" layer="95" font="vector" rot="R180"/>
-<attribute name="VALUE" x="116.332" y="73.025" size="1.778" layer="96" font="vector" rot="R180" align="top-left"/>
 </instance>
 <instance part="12V_LED" gate="G$1" x="111.76" y="58.42" smashed="yes" rot="R90">
 <attribute name="NAME" x="116.332" y="54.991" size="1.778" layer="95" font="vector" rot="R180"/>
-<attribute name="VALUE" x="116.332" y="60.325" size="1.778" layer="96" font="vector" rot="R180" align="top-left"/>
 </instance>
 <instance part="5.2V_LED" gate="G$1" x="111.76" y="45.72" smashed="yes" rot="R90">
 <attribute name="NAME" x="116.332" y="42.291" size="1.778" layer="95" font="vector" rot="R180"/>
-<attribute name="VALUE" x="116.332" y="47.625" size="1.778" layer="96" font="vector" rot="R180" align="top-left"/>
 </instance>
 <instance part="BMR480_POWERBRICK" gate="G$1" x="35.56" y="147.32" smashed="yes"/>
@@
 <net name="GND" class="0">
 <segment>
-<pinref part="BACKPLANE_CONN" gate="G$1" pin="P07"/>
-<wire x1="256.54" y1="149.86" x2="259.08" y2="149.86" width="0.1524" layer="91"/>
-<pinref part="BACKPLANE_CONN" gate="G$1" pin="P08"/>
-<wire x1="259.08" y1="149.86" x2="264.16" y2="149.86" width="0.1524" layer="91"/>
-<wire x1="256.54" y1="147.32" x2="259.08" y2="147.32" width="0.1524" layer="91"/>
-<wire x1="259.08" y1="147.32" x2="259.08" y2="149.86" width="0.1524" layer="91"/>
-<junction x="259.08" y="149.86"/>
-<label x="264.16" y="149.86" size="1.778" layer="95"/>
-</segment>
-<segment>
 <wire x1="20.32" y1="116.84" x2="20.32" y2="111.76" width="0.1524" layer="91"/>
 <wire x1="20.32" y1="111.76" x2="20.32" y2="109.22" width="0.1524" layer="91"/>
@@
 <label x="50.8" y="63.5" size="1.778" layer="95"/>
 </segment>
+<segment>
+<wire x1="256.54" y1="154.94" x2="259.08" y2="154.94" width="0.1524" layer="91"/>
+<wire x1="259.08" y1="154.94" x2="264.16" y2="154.94" width="0.1524" layer="91"/>
+<wire x1="256.54" y1="152.4" x2="259.08" y2="152.4" width="0.1524" layer="91"/>
+<wire x1="259.08" y1="152.4" x2="259.08" y2="154.94" width="0.1524" layer="91"/>
+<junction x="259.08" y="154.94"/>
+<label x="264.16" y="154.94" size="1.778" layer="95"/>
+<pinref part="BACKPLANE_CONN" gate="G$1" pin="P05"/>
+<pinref part="BACKPLANE_CONN" gate="G$1" pin="P06"/>
+</segment>
 </net>
 <net name="48V_GND" class="0">
@@
 </segment>
 <segment>
-<pinref part="D5" gate="G$1" pin="C"/>
+<pinref part="48V_LED" gate="G$1" pin="C"/>
 <wire x1="116.84" y1="71.12" x2="121.92" y2="71.12" width="0.1524" layer="91"/>
 <label x="121.92" y="71.12" size="1.778" layer="95"/>
@@
 <net name="N$9" class="0">
 <segment>
-<pinref part="D5" gate="G$1" pin="A"/>
+<pinref part="48V_LED" gate="G$1" pin="A"/>
 <pinref part="R8" gate="G$1" pin="2"/>
 <wire x1="109.22" y1="71.12" x2="104.14" y2="71.12" width="0.1524" layer="91"/>
@@
 </segment>
 <segment>
-<pinref part="BACKPLANE_CONN" gate="G$1" pin="P05"/>
-<wire x1="256.54" y1="154.94" x2="259.08" y2="154.94" width="0.1524" layer="91"/>
-<pinref part="BACKPLANE_CONN" gate="G$1" pin="P06"/>
-<wire x1="259.08" y1="154.94" x2="264.16" y2="154.94" width="0.1524" layer="91"/>
-<wire x1="256.54" y1="152.4" x2="259.08" y2="152.4" width="0.1524" layer="91"/>
-<wire x1="259.08" y1="152.4" x2="259.08" y2="154.94" width="0.1524" layer="91"/>
-<junction x="259.08" y="154.94"/>
-<label x="264.16" y="154.94" size="1.778" layer="95"/>
-</segment>
-<segment>
 <pinref part="U$6" gate="G$1" pin="VOUT+_5"/>
 <wire x1="121.92" y1="114.3" x2="132.08" y2="114.3" width="0.1524" layer="91"/>
@@
 <label x="157.48" y="45.72" size="1.778" layer="95"/>
 </segment>
-</net>
+<segment>
+<wire x1="256.54" y1="149.86" x2="259.08" y2="149.86" width="0.1524" layer="91"/>
+<wire x1="259.08" y1="149.86" x2="264.16" y2="149.86" width="0.1524" layer="91"/>
+<wire x1="256.54" y1="147.32" x2="259.08" y2="147.32" width="0.1524" layer="91"/>
+<wire x1="259.08" y1="147.32" x2="259.08" y2="149.86" width="0.1524" layer="91"/>
+<junction x="259.08" y="149.86"/>
+<label x="264.16" y="149.86" size="1.778" layer="95"/>
+<pinref part="BACKPLANE_CONN" gate="G$1" pin="P07"/>
+<pinref part="BACKPLANE_CONN" gate="G$1" pin="P08"/>
+</segment>
+</net>

Commit message: Minh Update 7
Parts:
- renumbered TRANS_REVERSE_VOLT_PROTEC to REVERSE_PROTECT
Changed lines of the file:
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@@
 <part name="D1" library="SparkFun-DiscreteSemi" library_urn="urn:adsk.eagle:library:514" deviceset="DIODE-ZENER" device="-BZT52C3V6S" package3d_urn="urn:adsk.eagle:package:38441/2" value="PZU15B3A,115"/>
 <part name="R4" library="SparkFun-Resistors" library_urn="urn:adsk.eagle:library:532" deviceset="RESISTOR" device="0603" package3d_urn="urn:adsk.eagle:package:41389018/1" value="1M"/>
-<part name="TRANS_REVERSE_VOLT_PROTEC" library="X15_Brickstribution" deviceset="TRANS_IRF1018ESTRLPBF" device="" package3d_urn="urn:adsk.eagle:package:25914649/1"/>
+<part name="REVERSE_PROTECT" library="X15_Brickstribution" deviceset="TRANS_IRF1018ESTRLPBF" device="" package3d_urn="urn:adsk.eagle:package:25914649/1"/>
 <part name="R8" library="SparkFun-Resistors" library_urn="urn:adsk.eagle:library:532" deviceset="0.1OHM" device="-0603-1/3W-1%" package3d_urn="urn:adsk.eagle:package:41389018/1" value="10k"/>
 <part name="R9" library="SparkFun-Resistors" library_urn="urn:adsk.eagle:library:532" deviceset="0.1OHM" device="-0603-1/3W-1%" package3d_urn="urn:adsk.eagle:package:41389018/1" value="500"/>
@@
 <attribute name="VALUE" x="184.404" y="160.02" size="1.778" layer="96" font="vector" rot="R90" align="top-center"/>
 </instance>
-<instance part="TRANS_REVERSE_VOLT_PROTEC" gate="G$1" x="193.04" y="144.78" smashed="yes" rot="R270">
+<instance part="REVERSE_PROTECT" gate="G$1" x="193.04" y="144.78" smashed="yes" rot="R270">
 <attribute name="NAME" x="193.04" y="139.7" size="1.778" layer="95" font="vector" rot="R270"/>
 <attribute name="VALUE" x="190.5" y="139.7" size="1.778" layer="96" font="vector" rot="R270"/>
@@
 <net name="48V_GND" class="0">
 <segment>
-<pinref part="TRANS_REVERSE_VOLT_PROTEC" gate="G$1" pin="S"/>
+<pinref part="REVERSE_PROTECT" gate="G$1" pin="S"/>
 <wire x1="187.96" y1="142.24" x2="175.26" y2="142.24" width="0.1524" layer="91"/>
 <pinref part="D1" gate="G$1" pin="A"/>
@@
 <wire x1="175.26" y1="149.86" x2="175.26" y2="152.4" width="0.1524" layer="91"/>
 <wire x1="175.26" y1="152.4" x2="182.88" y2="152.4" width="0.1524" layer="91"/>
-<pinref part="TRANS_REVERSE_VOLT_PROTEC" gate="G$1" pin="G"/>
+<pinref part="REVERSE_PROTECT" gate="G$1" pin="G"/>
 <wire x1="190.5" y1="149.86" x2="190.5" y2="152.4" width="0.1524" layer="91"/>
 <wire x1="190.5" y1="152.4" x2="182.88" y2="152.4" width="0.1524" layer="91"/>
@@
 <net name="GND_RAW" class="0">
 <segment>
-<pinref part="TRANS_REVERSE_VOLT_PROTEC" gate="G$1" pin="D"/>
+<pinref part="REVERSE_PROTECT" gate="G$1" pin="D"/>
 <wire x1="198.12" y1="142.24" x2="210.82" y2="142.24" width="0.1524" layer="91"/>
 <label x="198.12" y="142.24" size="1.778" layer="95"/>

Commit message: Minh Update 8
Parts:
- D1: value PZU15B3A,115 -> 3.6V
- R1: value 1k -> (none)
- R10: value 250 -> 0.1
- R2: value 3.32k -> (none)
- R3: value 150k -> 0.1
- R4: value 1M -> (none)
- R5: value 220k -> 0.1
- R8: value 10k -> 0.1
- R9: value 500 -> 0.1
Changed lines of the file:
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@@
 <part name="CIN2" library="SparkFun-Capacitors" library_urn="urn:adsk.eagle:library:510" deviceset="0.1UF" device="-0603-25V-(+80/-20%)" package3d_urn="urn:adsk.eagle:package:37414/1" value="0.1uF"/>
 <part name="C2" library="SparkFun-Capacitors" library_urn="urn:adsk.eagle:library:510" deviceset="0.1UF" device="-0603-25V-(+80/-20%)" package3d_urn="urn:adsk.eagle:package:37414/1" value="0.1uF"/>
-<part name="R1" library="SparkFun-Resistors" library_urn="urn:adsk.eagle:library:532" deviceset="RESISTOR" device="0603" package3d_urn="urn:adsk.eagle:package:41389018/1" value="1k"/>
-<part name="R2" library="SparkFun-Resistors" library_urn="urn:adsk.eagle:library:532" deviceset="RESISTOR" device="0603" package3d_urn="urn:adsk.eagle:package:41389018/1" value="3.32k"/>
+<part name="R1" library="SparkFun-Resistors" library_urn="urn:adsk.eagle:library:532" deviceset="RESISTOR" device="0603" package3d_urn="urn:adsk.eagle:package:41389018/1" value=" "/>
+<part name="R2" library="SparkFun-Resistors" library_urn="urn:adsk.eagle:library:532" deviceset="RESISTOR" device="0603" package3d_urn="urn:adsk.eagle:package:41389018/1" value=" "/>
 <part name="RADJ" library="SparkFun-Resistors" library_urn="urn:adsk.eagle:library:532" deviceset="RESISTOR" device="0603" package3d_urn="urn:adsk.eagle:package:41389018/1" value=" "/>
 <part name="40V_DIODE" library="X15-Conversion-Parts-Library" deviceset="CDBG520-G" device="" value="40V"/>
 <part name="FRAME1" library="SparkFun-Aesthetics" library_urn="urn:adsk.eagle:library:507" deviceset="FRAME-A4L" device=""/>
 <part name="BACKPLANE_CONN" library="X16_Power_Slab" deviceset="CONN_ET60T" device="" package3d_urn="urn:adsk.eagle:package:41523995/2"/>
-<part name="D1" library="SparkFun-DiscreteSemi" library_urn="urn:adsk.eagle:library:514" deviceset="DIODE-ZENER" device="-BZT52C3V6S" package3d_urn="urn:adsk.eagle:package:38441/2" value="PZU15B3A,115"/>
-<part name="R4" library="SparkFun-Resistors" library_urn="urn:adsk.eagle:library:532" deviceset="RESISTOR" device="0603" package3d_urn="urn:adsk.eagle:package:41389018/1" value="1M"/>
+<part name="D1" library="SparkFun-DiscreteSemi" library_urn="urn:adsk.eagle:library:514" deviceset="DIODE-ZENER" device="-BZT52C3V6S" package3d_urn="urn:adsk.eagle:package:38441/1" value="3.6V"/>
+<part name="R4" library="SparkFun-Resistors" library_urn="urn:adsk.eagle:library:532" deviceset="RESISTOR" device="0603" package3d_urn="urn:adsk.eagle:package:41389018/1" value=" "/>
 <part name="REVERSE_PROTECT" library="X15_Brickstribution" deviceset="TRANS_IRF1018ESTRLPBF" device="" package3d_urn="urn:adsk.eagle:package:25914649/1"/>
-<part name="R8" library="SparkFun-Resistors" library_urn="urn:adsk.eagle:library:532" deviceset="0.1OHM" device="-0603-1/3W-1%" package3d_urn="urn:adsk.eagle:package:41389018/1" value="10k"/>
-<part name="R9" library="SparkFun-Resistors" library_urn="urn:adsk.eagle:library:532" deviceset="0.1OHM" device="-0603-1/3W-1%" package3d_urn="urn:adsk.eagle:package:41389018/1" value="500"/>
-<part name="R10" library="SparkFun-Resistors" library_urn="urn:adsk.eagle:library:532" deviceset="0.1OHM" device="-0603-1/3W-1%" package3d_urn="urn:adsk.eagle:package:41389018/1" value="250"/>
+<part name="R8" library="SparkFun-Resistors" library_urn="urn:adsk.eagle:library:532" deviceset="0.1OHM" device="-0603-1/3W-1%" package3d_urn="urn:adsk.eagle:package:41389018/1" value="0.1"/>
+<part name="R9" library="SparkFun-Resistors" library_urn="urn:adsk.eagle:library:532" deviceset="0.1OHM" device="-0603-1/3W-1%" package3d_urn="urn:adsk.eagle:package:41389018/1" value="0.1"/>
+<part name="R10" library="SparkFun-Resistors" library_urn="urn:adsk.eagle:library:532" deviceset="0.1OHM" device="-0603-1/3W-1%" package3d_urn="urn:adsk.eagle:package:41389018/1" value="0.1"/>
 <part name="48V_LED" library="led" library_urn="urn:adsk.eagle:library:259" deviceset="LED" device="CHIPLED_0805" package3d_urn="urn:adsk.eagle:package:15821/2" value="48V"/>
 <part name="12V_LED" library="led" library_urn="urn:adsk.eagle:library:259" deviceset="LED" device="CHIPLED_0805" package3d_urn="urn:adsk.eagle:package:15821/2" value="12V"/>
@@
 <part name="48V_GND" library="X16-ExtraComponents" deviceset="TESTPOINT_5.04MM" device=""/>
 <part name="GND" library="X16-ExtraComponents" deviceset="TESTPOINT_5.04MM" device=""/>
-<part name="R3" library="SparkFun-Resistors" library_urn="urn:adsk.eagle:library:532" deviceset="0.1OHM" device="-0603-1/3W-1%" package3d_urn="urn:adsk.eagle:package:41389018/1" value="150k"/>
-<part name="R5" library="SparkFun-Resistors" library_urn="urn:adsk.eagle:library:532" deviceset="0.1OHM" device="-0603-1/3W-1%" package3d_urn="urn:adsk.eagle:package:41389018/1" value="220k"/>
+<part name="R3" library="SparkFun-Resistors" library_urn="urn:adsk.eagle:library:532" deviceset="0.1OHM" device="-0603-1/3W-1%" package3d_urn="urn:adsk.eagle:package:41389018/1" value="0.1"/>
+<part name="R5" library="SparkFun-Resistors" library_urn="urn:adsk.eagle:library:532" deviceset="0.1OHM" device="-0603-1/3W-1%" package3d_urn="urn:adsk.eagle:package:41389018/1" value="0.1"/>
 <part name="CIN1" library="X16_Power_Slab" deviceset="594D187X0016R2T" device=""/>
 </parts>
