File: X16_PowerSlab_V2.brd (EAGLE design)
At the start: 152.4 x 76.2 mm, 41 parts, among them J4 796636-6

Commit message: Minh update 4
Parts:
- CIN1: value 150uF -> 594D187X0016R2T; device X15-Conversion-Parts-Library:2917(7343-31-METRIC) -> X16_Power_Slab:CAP_X0016R2T_VIS
- moved R3 5.90 mm to (107.6, 33.0), flipped to the bottom, turned to 180 degrees
- moved R5 3.58 mm to (107.6, 35.0), flipped to the bottom, turned to 180 degrees
- moved CIN1 1.01 mm to (128.0, 44.1)
Connections:
- net GND: now also CIN1.2; no longer CIN1.-
- net VIN: now also CIN1.1; no longer CIN1.+
Routing:
- net GND: track 128.6 -> 122.4 mm, vias 27 -> 25
- net PMBUS_SA1: track 4.57 -> 3.78 mm
- net PMBUS_SA0: track 4.53 -> 3.78 mm
- net VIN: track 14.8 -> 15.3 mm
Other:
- board text added: "CIN1"
Changed lines of the file:
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@@
 <drawing>
 <settings>
-<setting alwaysvectorfont="no"/>
+<setting alwaysvectorfont="yes"/>
 <setting verticaltext="up"/>
 </settings>
@@
 <rectangle x1="77.8129" y1="66.8909" x2="78.1177" y2="66.9163" layer="21"/>
 <text x="0" y="-0.127" size="0.0508" layer="24" font="vector" rot="MR0">C:/Users/Minh/Downloads/crocs - Google Search.bmp</text>
+<text x="124.46" y="42.4942" size="1.016" layer="21" ratio="15" rot="R90">CIN1</text>
 </plain>
 <attributes>
@@
 <attribute name="VALUE" x="128.524" y="20.574" size="1.27" layer="28" rot="MR180" align="top-center"/>
 </element>
-<element name="CIN1" library="X15-Conversion-Parts-Library" package="2917(7343-31-METRIC)" package3d_urn="urn:adsk.eagle:package:25131320/3" value="150uF" x="127.254" y="43.434" smashed="yes" rot="R270">
-<attribute name="NAME" x="129.794" y="43.434" size="1.016" layer="25" ratio="15" rot="R270" align="bottom-center"/>
-<attribute name="VALUE" x="124.714" y="43.434" size="1.27" layer="27" rot="R270" align="top-center"/>
-</element>
 <element name="CR2" library="X16_Power_Slab" package="SDO_RBS2MM40CTR_ROM" value="RBS2MM40CTR" x="121.92" y="48.768" smashed="yes" rot="R90">
 <attribute name="COPYRIGHT" value="Copyright (C) 2023 Ultra Librarian. All rights reserved." x="121.92" y="48.768" size="1.778" layer="27" rot="R90" display="off"/>
@@
 <attribute name="VALUE" x="122.174" y="3.429" size="0.0254" layer="27"/>
 </element>
-<element name="R3" library="SparkFun-Resistors" library_urn="urn:adsk.eagle:library:532" package="0603" package3d_urn="urn:adsk.eagle:package:41389018/1" value="150k" x="104.267" y="28.1686" smashed="yes" rot="R270">
-<attribute name="NAME" x="105.029" y="28.1686" size="0.6096" layer="25" font="vector" ratio="20" rot="R270" align="bottom-center"/>
-<attribute name="PROD_ID" value="RES-15715" x="104.267" y="28.0162" size="1.778" layer="27" rot="R270" display="off"/>
-<attribute name="VALUE" x="103.505" y="28.1686" size="0.6096" layer="27" font="vector" ratio="20" rot="R270" align="top-center"/>
+<element name="R3" library="SparkFun-Resistors" library_urn="urn:adsk.eagle:library:532" package="0603" package3d_urn="urn:adsk.eagle:package:41389018/1" value="150k" x="107.6198" y="33.02" smashed="yes" rot="MR180">
+<attribute name="NAME" x="107.6198" y="32.258" size="1.016" layer="26" font="vector" ratio="15" rot="MR180" align="bottom-center"/>
+<attribute name="PROD_ID" value="RES-15715" x="107.7722" y="33.02" size="1.778" layer="28" rot="MR180" display="off"/>
+<attribute name="VALUE" x="107.6198" y="33.782" size="0.6096" layer="28" font="vector" ratio="20" rot="MR180" align="top-center"/>
+</element>
+<element name="R5" library="SparkFun-Resistors" library_urn="urn:adsk.eagle:library:532" package="0603" package3d_urn="urn:adsk.eagle:package:41389018/1" value="220k" x="107.6198" y="35.0266" smashed="yes" rot="MR180">
+<attribute name="NAME" x="107.6198" y="35.7632" size="1.016" layer="26" font="vector" ratio="15" rot="MR0" align="bottom-center"/>
+<attribute name="PROD_ID" value="RES-15715" x="107.7722" y="35.0266" size="1.778" layer="28" rot="MR180" display="off"/>
+<attribute name="VALUE" x="107.6198" y="35.7886" size="0.6096" layer="28" font="vector" ratio="20" rot="MR180" align="top-center"/>
 </element>
-<element name="R5" library="SparkFun-Resistors" library_urn="urn:adsk.eagle:library:532" package="0603" package3d_urn="urn:adsk.eagle:package:41389018/1" value="220k" x="105.791" y="31.9532" smashed="yes" rot="R270">
-<attribute name="NAME" x="106.553" y="31.9532" size="0.6096" layer="25" font="vector" ratio="20" rot="R270" align="bottom-center"/>
-<attribute name="PROD_ID" value="RES-15715" x="105.791" y="31.8008" size="1.778" layer="27" rot="R270" display="off"/>
-<attribute name="VALUE" x="105.029" y="31.9532" size="0.6096" layer="27" font="vector" ratio="20" rot="R270" align="top-center"/>
+<element name="CIN1" library="X16_Power_Slab" package="CAP_X0016R2T_VIS" value="594D187X0016R2T" x="128.016" y="44.0944" smashed="yes" rot="R270">
+<attribute name="COPYRIGHT" value="Copyright (C) 2023 Ultra Librarian. All rights reserved." x="128.016" y="44.0944" size="1.778" layer="27" rot="R270" display="off"/>
+<attribute name="MANUFACTURER_PART_NUMBER" value="594D187X0016R2T" x="128.016" y="44.0944" size="1.778" layer="27" rot="R270" display="off"/>
+<attribute name="MFR_NAME" value="Vishay" x="128.016" y="44.0944" size="1.778" layer="27" rot="R270" display="off"/>
+<attribute name="NAME" x="127.381" y="47.371" size="1.27" layer="27" ratio="6" rot="SR270"/>
+<attribute name="VALUE" x="127.381" y="45.8216" size="1.27" layer="27" ratio="6" rot="SR270"/>
 </element>
 </elements>
@@
 <contactref element="COUT5" pad="-"/>
 <contactref element="COUT6" pad="-"/>
-<contactref element="CIN1" pad="-"/>
 <polygon width="0.508" layer="16" isolate="0.762" thermals="no" rank="6">
 <vertex x="-1.778" y="80.772"/>
@@
 <wire x1="130.4544" y1="42.545" x2="130.4544" y2="52.74" width="0.508" layer="16"/>
 <contactref element="GND" pad="TP"/>
-<wire x1="127.254" y1="40.214" x2="122.092" y2="40.214" width="1.016" layer="1"/>
-<wire x1="122.092" y1="40.214" x2="121.92" y2="40.386" width="1.016" layer="1"/>
-<via x="121.92" y="40.386" extent="1-16" drill="1.27"/>
 <wire x1="98.044" y1="41.5798" x2="91.7702" y2="41.5798" width="1.016" layer="1"/>
 <wire x1="90.7202" y1="42.6298" x2="87.122" y2="42.6298" width="1.016" layer="1"/>
@@
 <via x="109.22" y="46.99" extent="1-16" drill="0.35"/>
 <via x="113.03" y="43.18" extent="1-16" drill="0.35"/>
-<via x="124.46" y="43.18" extent="1-16" drill="0.35"/>
 <via x="142.24" y="46.99" extent="1-16" drill="0.35"/>
 <via x="146.05" y="46.99" extent="1-16" drill="0.35"/>
@@
 <contactref element="R3" pad="2"/>
 <contactref element="R5" pad="2"/>
-<wire x1="105.791" y1="31.1032" x2="105.791" y2="27.2288" width="0.508" layer="1"/>
-<via x="105.791" y="27.2288" extent="1-16" drill="0.35"/>
-<wire x1="104.267" y1="27.3186" x2="105.7012" y2="27.3186" width="0.508" layer="1"/>
-<wire x1="105.7012" y1="27.3186" x2="105.791" y2="27.2288" width="0.508" layer="1"/>
+<contactref element="CIN1" pad="2"/>
+<wire x1="128.016" y1="41.8338" x2="123.4186" y2="41.8338" width="0.762" layer="1"/>
+<wire x1="123.4186" y1="41.8338" x2="123.3932" y2="41.8084" width="0.762" layer="1"/>
+<via x="123.3932" y="41.8084" extent="1-16" drill="0.8"/>
 </signal>
 <signal name="N$1">
@@
 <contactref element="BMR480_POWERBRICK" pad="PIN14"/>
 <contactref element="R5" pad="1"/>
-<wire x1="102.993" y1="35.0242" x2="105.0314" y2="35.0242" width="0.508" layer="1"/>
-<wire x1="105.791" y1="34.2646" x2="105.791" y2="32.8032" width="0.508" layer="1"/>
-<wire x1="105.0314" y1="35.0242" x2="105.791" y2="34.2646" width="0.508" layer="1"/>
+<wire x1="106.7698" y1="35.0266" x2="106.7674" y2="35.0242" width="0.762" layer="16"/>
+<wire x1="106.7674" y1="35.0242" x2="102.993" y2="35.0242" width="0.762" layer="16"/>
 </signal>
 <signal name="PMBUS_SA0">
 <contactref element="BMR480_POWERBRICK" pad="PIN15"/>
 <contactref element="R3" pad="1"/>
-<wire x1="102.993" y1="33.0176" x2="104.267" y2="31.7436" width="0.508" layer="1"/>
-<wire x1="104.267" y1="31.7436" x2="104.267" y2="29.0186" width="0.508" layer="1"/>
+<wire x1="106.7698" y1="33.02" x2="106.7674" y2="33.0176" width="0.762" layer="16"/>
+<wire x1="106.7674" y1="33.0176" x2="102.993" y2="33.0176" width="0.762" layer="16"/>
 </signal>
 <signal name="VIN">
 <contactref element="CIN2" pad="1"/>
 <contactref element="U$2" pad="PIN2"/>
-<contactref element="CIN1" pad="+"/>
 <contactref element="CR2" pad="1"/>
-<wire x1="132.9944" y1="45.7082" x2="132.9944" y2="45.466" width="0.508" layer="1"/>
-<wire x1="132.9944" y1="45.466" x2="132.9944" y2="44.5516" width="0.508" layer="1"/>
+<wire x1="132.9944" y1="45.7082" x2="132.9944" y2="44.5516" width="0.508" layer="1"/>
 <wire x1="132.9944" y1="44.5516" x2="133.096" y2="44.45" width="0.508" layer="1"/>
 <via x="133.096" y="44.45" extent="1-16" drill="0.35"/>
 <wire x1="133.096" y1="44.45" x2="133.096" y2="42.6466" width="0.508" layer="16"/>
 <wire x1="133.096" y1="42.6466" x2="132.9944" y2="42.545" width="0.508" layer="16"/>
-<wire x1="121.92" y1="46.6217" x2="121.9523" y2="46.654" width="1.27" layer="1"/>
-<wire x1="121.9523" y1="46.654" x2="127.254" y2="46.654" width="1.27" layer="1"/>
-<wire x1="132.16825" y1="46.0708" x2="132.3896" y2="46.0708" width="1.27" layer="1"/>
-<wire x1="132.3896" y1="46.0708" x2="132.9944" y2="45.466" width="1.27" layer="1"/>
-<wire x1="127.254" y1="46.654" x2="131.58505" y2="46.654" width="1.27" layer="1"/>
-<wire x1="131.58505" y1="46.654" x2="132.16825" y2="46.0708" width="1.27" layer="1"/>
+<contactref element="CIN1" pad="1"/>
+<wire x1="121.92" y1="46.6217" x2="127.4826" y2="46.6217" width="0.762" layer="1"/>
+<wire x1="127.4826" y1="46.6217" x2="127.7493" y2="46.6217" width="0.762" layer="1"/>
+<wire x1="127.7493" y1="46.6217" x2="128.016" y2="46.355" width="0.762" layer="1"/>
+<wire x1="132.9944" y1="45.7082" x2="128.3961" y2="45.7082" width="0.762" layer="1"/>
+<wire x1="128.3961" y1="45.7082" x2="127.4826" y2="46.6217" width="0.762" layer="1"/>
 </signal>
 </signals>

Commit message: Minh Update 5
Parts:
- removed D5: 48V, SparkFun-LED:LED-0805
- added 48V_LED: 48V, led:CHIPLED_0805
- 12V_LED, 5.2V_LED: device SparkFun-LED:LED-0805 -> led:CHIPLED_0805
- D1: value 3.6V -> PZU15B3A,115
- moved R9 7.31 mm to (82.6, 42.6), turned to 0 degrees
- moved R4 7.06 mm to (33.8, 18.2), turned to 180 degrees
- moved 12V_LED 1.07 mm to (86.9, 42.6), turned to 270 degrees
- moved COUT6 0.26 mm to (128.8, 18.0)
- moved 5.2V 0.13 mm to (133.8, 4.95)
- moved 5.2V_LED 0.05 mm to (146.9, 9.91), turned to 270 degrees
Connections:
- net 48V_GND: now also 48V_LED.C; no longer D5.C
- net 5.2V: now also BACKPLANE_CONN.P07_1, BACKPLANE_CONN.P07_10, BACKPLANE_CONN.P07_2, BACKPLANE_CONN.P07_3, BACKPLANE_CONN.P07_4, BACKPLANE_CONN.P07_5, BACKPLANE_CONN.P07_6, BACKPLANE_CONN.P07_7, BACKPLANE_CONN.P07_8, BACKPLANE_CONN.P07_9, BACKPLANE_CONN.P08_1, BACKPLANE_CONN.P08_10, BACKPLANE_CONN.P08_2, BACKPLANE_CONN.P08_3, BACKPLANE_CONN.P08_4, BACKPLANE_CONN.P08_5, BACKPLANE_CONN.P08_6, BACKPLANE_CONN.P08_7, BACKPLANE_CONN.P08_8, BACKPLANE_CONN.P08_9; no longer BACKPLANE_CONN.P05_1, BACKPLANE_CONN.P05_10, BACKPLANE_CONN.P05_2, BACKPLANE_CONN.P05_3, BACKPLANE_CONN.P05_4, BACKPLANE_CONN.P05_5, BACKPLANE_CONN.P05_6, BACKPLANE_CONN.P05_7, BACKPLANE_CONN.P05_8, BACKPLANE_CONN.P05_9, BACKPLANE_CONN.P06_1, BACKPLANE_CONN.P06_10, BACKPLANE_CONN.P06_2, BACKPLANE_CONN.P06_3, BACKPLANE_CONN.P06_4, BACKPLANE_CONN.P06_5, BACKPLANE_CONN.P06_6, BACKPLANE_CONN.P06_7, BACKPLANE_CONN.P06_8, BACKPLANE_CONN.P06_9
- net GND: now also BACKPLANE_CONN.P05_1, BACKPLANE_CONN.P05_10, BACKPLANE_CONN.P05_2, BACKPLANE_CONN.P05_3, BACKPLANE_CONN.P05_4, BACKPLANE_CONN.P05_5, BACKPLANE_CONN.P05_6, BACKPLANE_CONN.P05_7, BACKPLANE_CONN.P05_8, BACKPLANE_CONN.P05_9, BACKPLANE_CONN.P06_1, BACKPLANE_CONN.P06_10, BACKPLANE_CONN.P06_2, BACKPLANE_CONN.P06_3, BACKPLANE_CONN.P06_4, BACKPLANE_CONN.P06_5, BACKPLANE_CONN.P06_6, BACKPLANE_CONN.P06_7, BACKPLANE_CONN.P06_8, BACKPLANE_CONN.P06_9; no longer BACKPLANE_CONN.P07_1, BACKPLANE_CONN.P07_10, BACKPLANE_CONN.P07_2, BACKPLANE_CONN.P07_3, BACKPLANE_CONN.P07_4, BACKPLANE_CONN.P07_5, BACKPLANE_CONN.P07_6, BACKPLANE_CONN.P07_7, BACKPLANE_CONN.P07_8, BACKPLANE_CONN.P07_9, BACKPLANE_CONN.P08_1, BACKPLANE_CONN.P08_10, BACKPLANE_CONN.P08_2, BACKPLANE_CONN.P08_3, BACKPLANE_CONN.P08_4, BACKPLANE_CONN.P08_5, BACKPLANE_CONN.P08_6, BACKPLANE_CONN.P08_7, BACKPLANE_CONN.P08_8, BACKPLANE_CONN.P08_9
- net N$9: now also 48V_LED.A; no longer D5.A
Routing:
- net 12V: track 104.0 -> 87.1 mm
- net PMBUS_CTRL: track 68.9 -> 57.9 mm
- net GND: track 122.4 -> 113.4 mm, vias 25 -> 43
- net PMBUS_SDA: track 65.4 -> 56.7 mm
- net PMBUS_SALERT: track 62.5 -> 55.8 mm
- net PMBUS_SCL: track 61.3 -> 55.2 mm
- net 48V: track 43.5 -> 42.6 mm
- net N$7: track 6.49 -> 7.11 mm
